File: Dual_filter_common_mode_and_differential.sch (EAGLE design)
At the start: 23 parts

Commit message: Switched from CM-DIFF top CM-CM filtering
Parts:
- added C7, C8: 22nF, jqi_passives:C_MLCC_SMDCMLCC_0306
Connections:
- net -15V2: now also L7.3; no longer L7.1
- net COM2: now also L7.4; no longer L7.2
- net GND2: now also C7.1, C8.2, L6.2, L8.1; no longer L6.3, L8.4
- net N$10: now also L7.1, L8.4; no longer L7.3, L8.3
- net N$13: now also C8.1, L8.2; no longer L8.1
- net N$6: now also L6.3; no longer L6.4
- net N$7: now also L6.4; no longer L6.1
- net N$9: now also L7.2, L8.3; no longer L7.4, L8.2
- net V+2: now also C7.2, L6.1; no longer L6.2
Other:
- moved on the sheet: L6, L8
